Commit message: Small bug fixes

File: src/robot/robot_gazebo/objects/terrain.xacro (robot description, xacro)
@@ -49,5 +49,5 @@
     <xacro:if value="${'soft' == terrain}">
         <gazebo reference="ground_plane_link">
-            <material>Gazebo/Gold</material>
+            <material>Gazebo/Grass</material>
             <kp>5000</kp>
             <kd>100</kd>

Commit message: New terrain added: multi_terrains

File: src/robot/robot_gazebo/objects/terrain.xacro (robot description, xacro)
@@ -28,5 +28,5 @@
             </xacro:if>
             <xacro:if value="${'soft' == terrain}">
-                <material name="green">
+                <material name="gold">
                     <color rgba="0.8 0.8 0.0 1.0"/>
                 </material>

Commit message: The friction cones are displayed in RViz

File: src/robot/robot_gazebo/objects/terrain.xacro (robot description, xacro)
@@ -3,4 +3,5 @@
     <xacro:arg name="terrain" default="rigid"/>
     <xacro:property name="terrain" default="$(arg terrain)"/>
+    <xacro:property name="side" default="100"/>
     <gazebo>
         <static>true</static>
@@ -15,5 +16,5 @@
             <origin rpy="0 0 0" xyz="0 0 -1"/>
             <geometry>
-                <box size="100 100 2"/>
+                <box size="${side} ${side} 2"/>
             </geometry>
             <xacro:if value="${'rigid' == terrain}">
@@ -36,5 +37,5 @@
             <origin rpy="0 0 0" xyz="0 0 -1"/>
             <geometry>
-                <box size="100 100 2"/>
+                <box size="${side} ${side} 2"/>
             </geometry>
         </collision>
@@ -57,5 +58,5 @@
         <gazebo reference="ground_plane_link">
             <material>Gazebo/Gold</material>
-            <kp>1500</kp>
+            <kp>2000</kp>
             <kd>100</kd>
         </gazebo>

Commit message: The trotting planner uses the estimated terrain to correct the commanded base and feet height

File: src/robot/robot_gazebo/objects/terrain.xacro (robot description, xacro)
@@ -4,4 +4,10 @@
     <xacro:property name="terrain" default="$(arg terrain)"/>
     <xacro:property name="side" default="100"/>
+    <xacro:property name="roll"  default="0"/>
+    <xacro:property name="pitch" default="0"/>
+    <xacro:property name="yaw"   default="0"/>
+    <xacro:property name="x" default="0"/>
+    <xacro:property name="y" default="0"/>
+    <xacro:property name="z" default="-1"/>
     <gazebo>
         <static>true</static>
@@ -14,5 +20,5 @@
         </inertial>
         <visual>
-            <origin rpy="0 0 0" xyz="0 0 -1"/>
+            <origin rpy="${roll} ${pitch} ${yaw}" xyz="${x} ${y} ${z}"/>
             <geometry>
                 <box size="${side} ${side} 2"/>
@@ -35,5 +41,5 @@
         </visual>
         <collision>
-            <origin rpy="0 0 0" xyz="0 0 -1"/>
+            <origin rpy="${roll} ${pitch} ${yaw}" xyz="${x} ${y} ${z}"/>
             <geometry>
                 <box size="${side} ${side} 2"/>

Commit message: Can use a terrain generated from an heightmap + small changes

File: src/robot/robot_gazebo/objects/terrain.xacro (robot description, xacro)
@@ -14,9 +14,4 @@
     </gazebo>
     <link name="ground_plane_link">
-        <inertial>
-            <origin rpy="0 0 0" xyz="0 0 0"/>
-            <mass value="1"/>
-            <inertia ixx="1" ixy="0" ixz="0" iyy="1" iyz="0" izz="1"/>
-        </inertial>
         <visual>
             <origin rpy="${roll} ${pitch} ${yaw}" xyz="${x} ${y} ${z}"/>
@@ -47,4 +42,15 @@
         </collision>
     </link>
+    <joint name="ground_plane_link_to_ground_plane_link_inertia" type="fixed">
+        <parent link="ground_plane_link"/>
+        <child link="ground_plane_link_inertia"/>
+    </joint>
+    <link name="ground_plane_link_inertia">
+        <inertial>
+            <origin rpy="0 0 0" xyz="0 0 0"/>
+            <mass value="1"/>
+            <inertia ixx="1" ixy="0" ixz="0" iyy="1" iyz="0" izz="1"/>
+        </inertial>
+    </link>
     <xacro:if value="${'rigid' == terrain}">
         <gazebo reference="ground_plane_link">
